Commit message: Fix some merge errors.

File: boris_description/urdf/boris_description.xacro (robot description, xacro)
@@ -1,15 +1,12 @@
 <?xml version="1.0"?>
 <robot xmlns:xacro="http://www.ros.org/wiki/xacro" name="shark-v1">
+  <xacro:include filename="$(find shark_description)/urdf/shark.xacro" />
   <xacro:include filename="$(find sensors_description)/urdf/hokuyo.xacro" />
-  <xacro:include filename="$(find sensors_description)/urdf/sick_lms1xx.xacro" />
+  <xacro:include filename="$(find sensors_description)/urdf/sick_lms1xx.urdf.xacro" />
   <xacro:include filename="$(find sensors_description)/urdf/rgb_cam.xacro" />
-  <xacro:include filename="$(find sensors_description)/urdf/camera_turret.xacro" />
-  <xacro:include filename="$(find hector_models)/urdf/orbbec_astra2.xacro" />
-  <xacro:include filename="$(find hector_models)/gazebo/orbbec_astra2.gazebo.xacro" />
-  <xacro:include filename="$(find shark_description)/urdf/shark.xacro" />
-  <xacro:include filename="$(find sensors_description)/urdf/realsense_camera.urdf.xacro" />
+  <xacro:include filename="$(find sensors_description)/urdf/realsense_camera.xacro" />
   <xacro:include filename="$(find boris_head_description)/urdf/boris_head.urdf" />
-  <xacro:include filename="$(find boris_head_description)/urdf/control.urdf.xacro" />
-  <!-- <xacro:include filename="$(find boris_description)/ros2_control/shark_ros2_control.xacro" /> -->
+  <xacro:include filename="$(find interbotix_xsarm_descriptions)/urdf/wx200.urdf.xacro" />
+  <xacro:include filename="$(find shark_description)/ros2_control/shark_ros2_control.xacro" />
   <xacro:property name="base_width" value="0.336" />
   <xacro:property name="base_len" value="0.5" />
@@ -51,5 +48,5 @@
     </joint>
   </xacro:macro>
-  <xacro:sick_lms1xx robot_namespace="/lms1xx" />
+  <xacro:sick_lms_1xx name="sick" ros_topic="/scan" />
   <xacro:macro name="dorso" params="parent depth width height xyz rpy">
     <link name="dorso_link">
@@ -75,4 +72,5 @@
     </joint>
   </xacro:macro>
+    <!--32,5-->
   <xacro:macro name="arm_support" params="parent width height depth xyz rpy">
     <link name="arm_support_link">
@@ -101,14 +99,14 @@
     <child link="sick_mount_link" />
   </joint>
-  <!-- <joint name="dorso_head" type="fixed">
+  <joint name="dorso_head" type="fixed">
     <parent link="dorso_link" />
     <child link="head_root" />
     <origin xyz="0 0 ${dorso_height + 0.04}" rpy="0 0 0" />
-  </joint> -->
-  <!-- <joint name="arm_to_robot" type="fixed">
+  </joint>
+  <joint name="arm_to_robot" type="fixed">
     <origin xyz="0.1 0 ${arm_support_height/2}" rpy="0 0 0"/>
     <parent link="arm_support_link"/>
     <child link="wx200/base_link"/>
-  </joint> -->
+  </joint>
     <xacro:macro name="imu" params="parent xyz rpy">
     <link name="imu_link"/>
@@ -120,18 +118,4 @@
     </xacro:macro>
   <xacro:realsense_camera name="camera" parent="dorso_link" xyz="${dorso_len/2 + 0.05} 0 ${dorso_height + 0.053}" rpy="0 0 0"/>
-  <xacro:realsense_camera name="camera" parent="dorso_link">
-    <origin xyz="${dorso_len/2 + 0.05} 0 ${dorso_height + 0.053}" rpy="0 0 ${3.14/8}" />
-  </xacro:realsense_camera>
-  <xacro:realsense_gazebo />
-  <xacro:add_optical_frame name="camera_link" />
-  <xacro:camera_turret parent="dorso_link" name="camera_turret">
-    <origin xyz="${dorso_len/2 + 0.05} 0 ${dorso_height + 0.053}" rpy="0 0 ${3.14/8}" />
-  </xacro:camera_turret>
-  <xacro:orbbec_astra2 name="top_camera">
-    <parent link="camera_turret_tilt_link"/>
-    <origin rpy="0 0 -${M_PI/6}" xyz="0.06705 0 -0.00425"/>
-  </xacro:orbbec_astra2>
-  <xacro:orbbec_astra2_gazebo name="top_camera" semantic_segmentation="false"/>
-  <xacro:orbbec_astra2_gazebo name="top_camera"/>
   <xacro:dorso parent="base_link" depth="${dorso_len}" width="${dorso_width}" height="${dorso_height}" xyz="${-base_len/2 + (dorso_len/2)} 0 ${base_height/2}" rpy="0 0 0"/>
   <xacro:arm_support parent="dorso_link" width="${arm_support_width}" height="${arm_support_height}" depth="${arm_support_len}" xyz="${dorso_len/2 + arm_support_len/2} 0 ${arm_z_position}" rpy="0 0 0"/>
@@ -144,10 +128,2 @@
   <xacro:shark_base/>  <!-- isso aq n existe mais, a gente reverteu as mudanças do luis que transformavam aquilo tudo em um macro q n ta aparecendo mais -->
 </robot>
-  <xacro:imu parent="base_link" xyz="-0.01 0 ${0.02 - base_height/2}" rpy="-0.014161 -0.0203861 0" />
-  <gazebo reference="dorso_link">
-    <material>Gazebo/DarkGray</material>
-  </gazebo>
-  <gazebo reference="arm_support_link">
-    <material>Gazebo/DarkGray</material>
-  </gazebo>
-</robot>

File: sensors_description/urdf/realsense_camera.xacro (robot description, xacro)
@@ -2,81 +2,6 @@
 <robot name="realsense_rgbd" xmlns:xacro="http://www.ros.org/wiki/xacro">
   <xacro:property name="M_PI" value="3.1415926535897931"/>
-  <xacro:macro name="add_optical_frame" params="name">
-		<joint name="${name}_optical_joint" type="fixed">
-			<origin xyz="0 0 0" rpy="0.0 0.0 0.0" />
-			<parent link="${name}" />
-			<child link="${name}_optical_frame"/>
-		</joint>
-		<link name="${name}_optical_frame" />
-	</xacro:macro>
-  <xacro:macro name="realsense_gazebo">
-		<gazebo reference="camera_link_optical_frame">
-			<sensor type="camera" name="realsense">
-				<always_on>true</always_on>
-				<visualize>true</visualize>
-				<update_rate>15</update_rate>
-				<gz_frame_id>camera_link_optical_frame</gz_frame_id>
-				<camera>
-					<optical_frame_id>camera_link_optical_frame</optical_frame_id>
-					<horizontal_fov>1.047</horizontal_fov>
-					<image>
-						<width>640</width>
-						<height>480</height>
-					</image>
-					<depth_camera>
-						<clip>
-							<near>0.1</near>
-							<far>10.0</far>
-						</clip>
-					</depth_camera>
-					<noise>
-						<type>gaussian</type>
-						<mean>0.0</mean>
-						<stddev>0.01</stddev>
-					</noise>
-				</camera>
-                <plugin name="realsense_camera_plugin" filename="libgazebo_ros_camera.so">
-                    <ros>
-                    <remapping>image_raw:=/realsense/image_color/raw</remapping>
-                    <remapping>camera_info:=/realsense/image_color/camera_info</remapping>
-                    <frame_name>camera_link_optical_frame</frame_name>
-                    </ros>
-                </plugin>
-			</sensor>
-            <sensor type="depth" name="realsense_depth">
-				<always_on>true</always_on>
-				<visualize>true</visualize>
-				<update_rate>15</update_rate>
-				<gz_frame_id>camera_link_optical_frame</gz_frame_id>
-				<camera>
-					<optical_frame_id>camera_link_optical_frame</optical_frame_id>
-					<horizontal_fov>1.047</horizontal_fov>
-					<image>
-						<width>640</width>
-						<height>480</height>
-					</image>
-					<depth_camera>
-						<clip>
-							<near>0.1</near>
-							<far>10.0</far>
-						</clip>
-					</depth_camera>
-					<noise>
-						<type>gaussian</type>
-						<mean>0.0</mean>
-						<stddev>0.01</stddev>
-					</noise>
-				</camera>
-                <plugin name="realsense_camera_plugin" filename="libgazebo_ros_camera.so">
-                    <ros>
-                    <remapping>image_raw:=/realsense/image_depth/raw</remapping>
-                    <remapping>camera_info:=/realsense/image_depth/camera_info</remapping>
-                    <frame_name>camera_link_optical_frame</frame_name>
-                    </ros>
-                </plugin>
-			</sensor>
-		</gazebo>
-	</xacro:macro>
-  <xacro:macro name="realsense_camera" params="name parent *origin">
+  <xacro:macro name="realsense_camera" params="name parent xyz rpy">
+      <!-- @TODO: GABIARRA PRA GIRAR A CAMERA -->
       <link name="head_pan_link_static">
           <inertial>
@@ -206,19 +131,7 @@
           <axis xyz="0 0 0"/>
       </joint>
-      <ros2_control name="head_hardware_interface" type="system">
-    <hardware>
-      <plugin>gazebo_ros2_control/GazeboSystem</plugin>
-    </hardware>
-    <joint name="head_pan_joint">
-      <command_interface name="position">
-      </command_interface>
-      <state_interface name="position"/>
-    </joint>
-    <joint name="head_tilt_joint">
-      <command_interface name="position">
-      </command_interface>
-      <state_interface name="position"/>
-    </joint>
-  </ros2_control>
+      <!-- <xacro:sensor_d435 parent="head_tilt_link" use_nominal_extrinsics="false" add_plug="false" use_mesh="true">
+          <origin xyz="0.06705 0 -0.00425" rpy="0 0 0"/>
+      </xacro:sensor_d435> -->
   </xacro:macro>
 </robot>

File: shark_description/urdf/shark_description.xacro (robot description, xacro)
@@ -10,6 +10,4 @@
   <xacro:property name="wheel_joint_offset" value="0.0" />
   <xacro:property name="caster_height" value="0.07" />
-  <xacro:property name="caster_wheel_joint_offset" value="0.0" />
-  <xacro:property name="caster_wheel_radius" value="0.02" />
   <xacro:macro name="box_inertia" params="m w h d">
     <inertial>
@@ -18,25 +16,4 @@
     </inertial>
   </xacro:macro>
-  <link name="base_footprint">
-  </link>
-  <link name="base_link">
-    <xacro:box_inertia m="1" w="${base_len}" h="${base_width}" d="0.01"/>
-    <visual>
-      <material name="lightgray"/>
-      <geometry>
-        <box size="${base_len} ${base_width} ${base_height}"/>
-      </geometry>
-    </visual>
-    <collision>
-      <geometry>
-        <box size="${base_len} ${base_width} ${base_height}"/>
-      </geometry>
-    </collision>
-  </link>
-  <joint name="base_link_joint" type="fixed">
-    <origin xyz="0 0 ${base_height/2 + caster_height}" rpy="0 0 0" />
-    <parent link="base_footprint"/>
-    <child link="base_link" />
-  </joint>
   <xacro:macro name="cylinder_inertia" params="m r h">
     <inertial>
@@ -62,5 +39,5 @@
       <xacro:cylinder_inertia m="10" r="${wheel_radius}" h="0.05"/>
     </link>
-    <joint name="${prefix}_wheel_joint" type="continuous">
+    <joint name="${prefix}_wheel" type="continuous">
       <axis xyz="0 1 0" rpy="0 0 0" />
       <parent link="base_link"/>
@@ -75,25 +52,27 @@
     </inertial>
   </xacro:macro>
-   <link name="caster_wheel">
-     <visual>
-       <material name="darkgray"/>
-      <origin xyz="0 0 0" rpy="0 0 0"/>
-      <geometry>
-        <sphere radius="${caster_wheel_radius}"/>
-      </geometry>
-    </visual>
-    <collision>
-      <origin xyz="0 0 0" rpy="0 0 0"/>
-      <geometry>
-        <sphere radius="${caster_wheel_radius}"/>
-      </geometry>
-    </collision>
-    <xacro:sphere_inertia m="5" r="${caster_wheel_radius}"/>
-  </link>
-  <joint name="caster_wheel_joint" type="continuous">
-    <axis xyz="0 1 0" rpy="0 0 0" />
-    <parent link="base_link"/>
-    <child link="caster_wheel"/>
-    <origin xyz="${(base_len/2) - caster_wheel_joint_offset} 0 ${(caster_wheel_radius - caster_height) - base_height/2}" rpy="0 0 0"/>
-  </joint>
+  <xacro:macro name="shark_base">
+    <link name="base_footprint"/>
+    <link name="base_link">
+      <xacro:box_inertia m="1" w="${base_len}" h="${base_width}" d="0.01" />
+      <visual>
+        <material name="lightgray" />
+        <geometry>
+          <box size="${base_len} ${base_width} ${base_height}" />
+        </geometry>
+      </visual>
+      <collision>
+        <geometry>
+          <box size="${base_len} ${base_width} ${base_height}" />
+        </geometry>
+      </collision>
+    </link>
+    <joint name="base_link_joint" type="fixed">
+      <origin xyz="0 0 ${base_height/2 + caster_height}" rpy="0 0 0" />
+      <parent link="base_footprint" />
+      <child link="base_link" />
+    </joint>
+    <xacro:wheel prefix="left" reflect="1" />
+    <xacro:wheel prefix="right" reflect="-1" />
+  </xacro:macro>
 </robot>

Commit message: refactor: remove interbotix arm control and static transform publisher; add conditional arm attachment in URDF

File: boris_description/urdf/boris_description.xacro (robot description, xacro)
@@ -26,4 +26,5 @@
   <xacro:arg name="arm_z_position" default="0.34"/>
   <xacro:property name="arm_z_position" value="$(arg arm_z_position)" />
+  <xacro:arg name="use_arm" default="true"/>
   <xacro:macro name="box_inertia" params="m w h d">
     <inertial>
@@ -104,9 +105,18 @@
     <origin xyz="0 0 ${dorso_height + 0.04}" rpy="0 0 0" />
   </joint> -->
-  <!-- <joint name="arm_to_robot" type="fixed">
-    <origin xyz="0.1 0 ${arm_support_height/2}" rpy="0 0 0"/>
-    <parent link="arm_support_link"/>
-    <child link="wx200/base_link"/>
-  </joint> -->
+  <!-- wx200 arm attachment. The arm's own model/TF/hardware come from the Interbotix stack
+       (xsarm_moveit.launch.py), whose namespaced robot_state_publisher owns the wx200/* subtree.
+       Here we only declare the attach point + a real fixed joint, so the BORIS<->arm connection
+       lives in the URDF instead of a runtime static_transform_publisher. We deliberately do NOT
+       include wx200.urdf.xacro: doing so would double-publish wx200/* on the global /tf and drag
+       the interbotix <ros2_control> block into the BORIS base controller_manager. -->
+  <xacro:if value="$(arg use_arm)">
+    <link name="wx200/base_link"/>
+    <joint name="arm_to_robot" type="fixed">
+      <origin xyz="0.1 0 ${arm_support_height/2}" rpy="0 0 0"/>
+      <parent link="arm_support_link"/>
+      <child link="wx200/base_link"/>
+    </joint>
+  </xacro:if>
     <xacro:macro name="imu" params="parent xyz rpy">
     <link name="imu_link"/>

Commit message: feat: add arm_z_position argument and adjust femtobolt camera mounting parameters

File: boris_description/urdf/boris_description.xacro (robot description, xacro)
@@ -128,5 +128,5 @@
     </xacro:macro>
   <!-- TODO: re-measure dorso_link -> neck pan axis if the neck/camera moved -->
-  <xacro:femtobolt_camera name="camera" parent="dorso_link" xyz="${dorso_len/2 + 0.05} 0 ${dorso_height + 0.053}" rpy="0 0 0"/>
+  <xacro:femtobolt_camera name="camera" parent="dorso_link" xyz="${dorso_len/2 + 0.042} 0 ${dorso_height}" rpy="0 0 0"/>
   <xacro:dorso parent="base_link" depth="${dorso_len}" width="${dorso_width}" height="${dorso_height}" xyz="${-base_len/2 + (dorso_len/2)} 0 ${base_height/2}" rpy="0 0 0"/>
   <xacro:arm_support parent="dorso_link" width="${arm_support_width}" height="${arm_support_height}" depth="${arm_support_len}" xyz="${dorso_len/2 + arm_support_len/2} 0 ${arm_z_position}" rpy="0 0 0"/>

File: sensors_description/urdf/femtobolt_camera.xacro (robot description, xacro)
@@ -17,5 +17,5 @@
       - femtobolt_size       : outer box of the Femto Bolt body (x=depth y=width z=height)
   -->
-  <xacro:property name="femtobolt_mount_xyz" value="0.05 0 -0.05"/>   <!-- TODO measure: head_tilt_link -> camera_link -->
+  <xacro:property name="femtobolt_mount_xyz" value="0.05 0 -0.04"/>   <!-- TODO measure: head_tilt_link -> camera_link -->
   <xacro:property name="femtobolt_mount_rpy" value="${M_PI} 0 0"/>          <!-- 180° roll: corrects the camera_color_optical_frame being rolled 180° about the viewing axis (Femto Bolt mounted/published inverted). Use "0 0 0" if not needed. -->
   <xacro:property name="femtobolt_size"      value="0.026 0.0996 0.0395"/>   <!-- TODO measure: Femto Bolt body x y z -->
@@ -96,5 +96,5 @@
       </link>
       <joint name="head_tilt_joint_static" type="fixed">
-          <origin rpy="0 0 0" xyz="0 0 0.05"/>
+          <origin rpy="0 0 0" xyz="0 0 0.057"/>
           <parent link="head_pan_link_static"/>
           <child link="head_tilt_link_static"/>
@@ -103,5 +103,5 @@
       </joint>
       <joint name="head_tilt_joint" type="revolute">
-          <origin rpy="0 0 0" xyz="0 0 0.05"/>
+          <origin rpy="0 0 0" xyz="0 0 0.057"/>
           <parent link="head_pan_link"/>
           <child link="head_tilt_link"/>

Commit message: fix: adjust arm_z_position and femtobolt_mount_xyz for improved alignment

File: boris_description/urdf/boris_description.xacro (robot description, xacro)
@@ -24,5 +24,5 @@
   <xacro:property name="arm_support_len" value="0.325" />
   <xacro:property name="arm_support_height" value="0.047" />
-  <xacro:arg name="arm_z_position" default="0.34"/>
+  <xacro:arg name="arm_z_position" default="0.315"/>
   <xacro:property name="arm_z_position" value="$(arg arm_z_position)" />
   <xacro:arg name="use_arm" default="true"/>

File: sensors_description/urdf/femtobolt_camera.xacro (robot description, xacro)
@@ -17,5 +17,5 @@
       - femtobolt_size       : outer box of the Femto Bolt body (x=depth y=width z=height)
   -->
-  <xacro:property name="femtobolt_mount_xyz" value="0.05 0 -0.04"/>   <!-- TODO measure: head_tilt_link -> camera_link -->
+  <xacro:property name="femtobolt_mount_xyz" value="0.05 0 0.04"/>   <!-- TODO measure: head_tilt_link -> camera_link -->
   <xacro:property name="femtobolt_mount_rpy" value="0 0 0"/>          <!-- 180° roll: corrects the camera_color_optical_frame being rolled 180° about the viewing axis (Femto Bolt mounted/published inverted). Use "0 0 0" if not needed. -->
   <xacro:property name="femtobolt_size"      value="0.026 0.0996 0.0395"/>   <!-- TODO measure: Femto Bolt body x y z -->
