Commit message: fix sensors to allow simulation

File: boris_description/urdf/boris_description.xacro (robot description, xacro)
@@ -7,5 +7,5 @@
   <xacro:include filename="$(find sensors_description)/urdf/realsense_camera.xacro" />
   <!-- <xacro:include filename="$(find boris_head_description)/urdf/boris_head.urdf" /> -->
-  <!-- <xacro:include filename="$(find interbotix_xsarm_descriptions)/urdf/wx200.urdf.xacro" /> -->
+  <xacro:include filename="$(find interbotix_xsarm_descriptions)/urdf/wx200.urdf.xacro" />
   <!-- <xacro:include filename="$(find boris_description)/ros2_control/shark_ros2_control.xacro" /> -->
   <xacro:property name="base_width" value="0.336" />
@@ -104,9 +104,9 @@
     <origin xyz="0 0 ${dorso_height + 0.04}" rpy="0 0 0" />
   </joint> -->
-  <!-- <joint name="arm_to_robot" type="fixed">
+  <joint name="arm_to_robot" type="fixed">
     <origin xyz="0.1 0 ${arm_support_height/2}" rpy="0 0 0"/>
     <parent link="arm_support_link"/>
     <child link="wx200/base_link"/>
-  </joint> -->
+  </joint>
     <xacro:macro name="imu" params="parent xyz rpy">
     <link name="imu_link"/>

File: sensors_description/urdf/hokuyo.xacro (robot description, xacro)
@@ -1,13 +1,6 @@
 <?xml version="1.0"?>
-<robot name="sensor_hokuyo"
-  xmlns:xacro="http://ros.org/wiki/xacro">
+<robot name="sensor_hokuyo" xmlns:xacro="http://ros.org/wiki/xacro">
   <xacro:macro name="sensor_hokuyo" params="parent xyz rpy name">
     <link name="hokuyo_${name}_link">
-      <!--collision>
-        <origin xyz="0 0 0" rpy="0 0 0"/>
-        <geometry>
-          <box size="0.01 0.01 0.01"/>
-        </geometry>
-      </collision-->
       <visual>
         <origin xyz="0 0 0" rpy="0 0 0"/>
@@ -23,24 +16,24 @@
     </link>
     <joint name="hokuyo_${name}_joint" type="fixed">
-      <!--<axis xyz="0 0 1" />-->
       <origin xyz="${xyz}" rpy="${rpy}"/>
       <parent link="${parent}"/>
       <child link="hokuyo_${name}_link"/>
     </joint>
-    <!-- Hokuyo sensor for simulation -->
-    <xacro:sim_laser_range_finder/>
+    <xacro:sim_laser_range_finder name="${name}"/>
   </xacro:macro>
-  <!-- ULM-30LX Hokuyo Laser Range Finder -->
-  <xacro:macro name="sim_laser_range_finder">
+  <xacro:macro name="sim_laser_range_finder" params="name">
     <gazebo reference="hokuyo_${name}_link">
-      <sensor type="ray" name="head_hokuyo_sensor">
+      <sensor type="gpu_lidar" name="hokuyo_${name}_sensor">
         <pose>0 0 0 0 0 0</pose>
-        <visualize>false</visualize>
-        <update_rate>40</update_rate>
+        <topic>scan_${name}</topic>
+        <ignition_frame_id>hokuyo_${name}_link</ignition_frame_id>
+        <always_on>true</always_on>
+        <visualize>true</visualize>
+        <update_rate>20</update_rate>
         <ray>
           <scan>
             <horizontal>
               <samples>683</samples>
-              <resolution>0.3515625</resolution>
+              <resolution>1</resolution>
               <min_angle>-2.0943</min_angle>
               <max_angle>2.0943</max_angle>
@@ -54,17 +47,8 @@
           <noise>
             <type>gaussian</type>
-            <!-- Noise parameters based on published spec for Hokuyo laser
-               achieving "+-30mm" accuracy at range < 10m.  A mean of 0.0m and
-               stddev of 0.01m will put 99.7% of samples within 0.03m of the true
-               reading. -->
             <mean>0.0</mean>
             <stddev>0.01</stddev>
           </noise>
         </ray>
-        <plugin name="gazebo_ros_head_hokuyo_controller" filename="libgazebo_ros_laser.so">
-          <topicName>scan2</topicName>
-          <frameName>hokuyo_${name}_link</frameName>
-          <robotNamespace>/</robotNamespace>
-        </plugin>
       </sensor>
     </gazebo>

File: sensors_description/urdf/sick_lms1xx.urdf.xacro (robot description, xacro)
@@ -1,7 +1,4 @@
 <?xml version="1.0"?>
-<robot xmlns:controller="http://playerstage.sourceforge.net/gazebo/xmlschema/#controller"
-  xmlns:interface="http://playerstage.sourceforge.net/gazebo/xmlschema/#interface"
-  xmlns:sensor="http://playerstage.sourceforge.net/gazebo/xmlschema/#sensor"
-  xmlns:xacro="http://ros.org/wiki/xacro">
+<robot xmlns:xacro="http://ros.org/wiki/xacro">
   <xacro:macro name="sick_lms_1xx" params="name ros_topic gaussian_noise:=0.006">
     <xacro:sick_lms_1 name="${name}" ros_topic="${ros_topic}"
@@ -15,5 +12,5 @@
           <mesh filename="package://sensors_description/meshes/sick-lms1xx.stl"/>
         </geometry>
-        <material name="grey" >
+        <material name="grey">
           <color rgba="0 0 1 1" />
         </material>
@@ -49,10 +46,11 @@
   <xacro:macro name="sick_lms_1_laser_gazebo_v0" params="name link ros_topic update_rate min_angle max_angle min_range max_range gaussian_noise">
     <gazebo reference="${link}">
-      <material value="Gazebo/Blue" />
-      <sensor type="ray" name="${name}">
+      <sensor type="gpu_lidar" name="${name}">
         <always_on>true</always_on>
         <update_rate>${update_rate}</update_rate>
         <pose>0 0 0 0 0 0</pose>
-        <visualize>false</visualize>
+        <topic>scan</topic>
+        <ignition_frame_id>${link}</ignition_frame_id>
+        <visualize>true</visualize>
         <ray>
           <scan>
@@ -75,8 +73,4 @@
           </noise>
         </ray>
-        <plugin name="gazebo_ros_${name}_controller" filename="libgazebo_ros_laser.so">
-          <topicName>${ros_topic}</topicName>
-          <frameName>${link}</frameName>
-        </plugin>
       </sensor>
     </gazebo>

File: shark_description/ros2_control/shark_ros2_control.xacro (robot description, xacro)
@@ -1,21 +1,102 @@
 <?xml version="1.0"?>
-<robot>
+<robot xmlns:xacro="http://www.ros.org/wiki/xacro">
+  <xacro:arg name="use_sim" default="false"/>
   <ros2_control name="shark" type="system">
     <hardware>
-      <plugin>hoverboard_driver/hoverboard_driver</plugin>
-      <param name="wheel_radius">0.0775</param>
-      <param name="max_velocity">1.0</param>
-      <param name="device">/dev/ttySHARK</param>
+      <xacro:if value="$(arg use_sim)">
+        <plugin>gz_ros2_control/GazeboSimSystem</plugin>
+      </xacro:if>
+      <xacro:unless value="$(arg use_sim)">
+        <plugin>hoverboard_driver/hoverboard_driver</plugin>
+        <param name="wheel_radius">0.0775</param>
+        <param name="max_velocity">1.0</param>
+        <param name="device">/dev/ttySHARK</param>
+      </xacro:unless>
     </hardware>
     <joint name="left_wheel_joint">
-      <command_interface name="velocity"/>
+      <command_interface name="velocity">
+        <xacro:if value="$(arg use_sim)">
+          <param name="min">-1</param>
+          <param name="max">1</param>
+        </xacro:if>
+      </command_interface>
       <state_interface name="position"/>
       <state_interface name="velocity"/>
     </joint>
     <joint name="right_wheel_joint">
-      <command_interface name="velocity"/>
+      <command_interface name="velocity">
+        <xacro:if value="$(arg use_sim)">
+          <param name="min">-1</param>
+          <param name="max">1</param>
+        </xacro:if>
+      </command_interface>
       <state_interface name="position"/>
       <state_interface name="velocity"/>
     </joint>
+    <xacro:if value="$(arg use_sim)">
+      <joint name="waist">
+        <command_interface name="position"/>
+        <state_interface name="position">
+          <param name="initial_value">0.0</param>
+        </state_interface>
+        <state_interface name="velocity"/>
+      </joint>
+      <joint name="shoulder">
+        <command_interface name="position"/>
+        <state_interface name="position">
+          <param name="initial_value">0.0</param>
+        </state_interface>
+        <state_interface name="velocity"/>
+      </joint>
+      <joint name="elbow">
+        <command_interface name="position"/>
+        <state_interface name="position">
+          <param name="initial_value">0.0</param>
+        </state_interface>
+        <state_interface name="velocity"/>
+      </joint>
+      <joint name="wrist_angle">
+        <command_interface name="position"/>
+        <state_interface name="position">
+          <param name="initial_value">0.0</param>
+        </state_interface>
+        <state_interface name="velocity"/>
+      </joint>
+      <joint name="wrist_rotate">
+        <command_interface name="position"/>
+        <state_interface name="position">
+          <param name="initial_value">0.0</param>
+        </state_interface>
+        <state_interface name="velocity"/>
+      </joint>
+      <joint name="gripper">
+        <command_interface name="position"/>
+        <state_interface name="position">
+          <param name="initial_value">0.0</param>
+        </state_interface>
+        <state_interface name="velocity"/>
+      </joint>
+      <joint name="left_finger">
+        <command_interface name="position"/>
+        <state_interface name="position">
+          <param name="initial_value">0.02</param>
+        </state_interface>
+        <state_interface name="velocity"/>
+      </joint>
+      <joint name="right_finger">
+        <command_interface name="position"/>
+        <state_interface name="position">
+          <param name="initial_value">-0.02</param>
+        </state_interface>
+        <state_interface name="velocity"/>
+      </joint>
+    </xacro:if>
   </ros2_control>
+  <xacro:if value="$(arg use_sim)">
+    <gazebo>
+      <plugin filename="gz_ros2_control-system" name="gz_ros2_control::GazeboSimROS2ControlPlugin">
+        <parameters>$(find shark_description)/config/shark_controllers_sim.yaml</parameters>
+      </plugin>
+    </gazebo>
+  </xacro:if>
 </robot>

File: shark_description/urdf/shark_description.xacro (robot description, xacro)
@@ -19,5 +19,11 @@
     <inertial>
       <mass value="${m}"/>
-      <inertia ixx="${m*(3*r*r+h*h)/12}" ixy = "0" ixz = "0" iyy="${m*(3*r*r+h*h)/12}" iyz = "0" izz="${m*r*r/2}"/>
+      <inertia ixx="${m*(3*r*r+h*h)/12}" ixy="0" ixz="0" iyy="${m*(3*r*r+h*h)/12}" iyz="0" izz="${m*r*r/2}"/>
+    </inertial>
+  </xacro:macro>
+  <xacro:macro name="sphere_inertia" params="m r">
+    <inertial>
+      <mass value="${m}"/>
+      <inertia ixx="${2.0*m*(r*r)/5.0}" ixy="0.0" ixz="0.0" iyy="${2.0*m*(r*r)/5.0}" iyz="0.0" izz="${2.0*m*(r*r)/5.0}"/>
     </inertial>
   </xacro:macro>
@@ -25,5 +31,5 @@
     <link name="${prefix}_wheel">
       <visual>
-	      <material name="darkgray"/>
+        <material name="darkgray"/>
         <origin xyz="0 0 0" rpy="${pi/2} 0 0"/>
         <geometry>
@@ -39,5 +45,5 @@
       <xacro:cylinder_inertia m="10" r="${wheel_radius}" h="0.05"/>
     </link>
-    <joint name="${prefix}_wheel" type="continuous">
+    <joint name="${prefix}_wheel_joint" type="continuous">
       <axis xyz="0 1 0" rpy="0 0 0" />
       <parent link="base_link"/>
@@ -46,9 +52,34 @@
     </joint>
   </xacro:macro>
-  <xacro:macro name="sphere_inertia" params="m r">
-    <inertial>
-      <mass value="${m}"/>
-      <inertia ixx="${2.0*m*(r*r)/5.0}" ixy="0.0" ixz="0.0" iyy="${2.0*m*(r*r)/5.0}" iyz="0.0" izz="${2.0*m*(r*r)/5.0}"/>
-    </inertial>
+  <!-- Macro das rodas de apoio (caster) frontal e traseira para nivelar o Boris -->
+  <xacro:macro name="caster_wheel" params="prefix x_offset">
+    <link name="${prefix}_caster_wheel">
+      <visual>
+        <material name="darkgray"/>
+        <origin xyz="0 0 0" rpy="0 0 0"/>
+        <geometry>
+          <sphere radius="${caster_height/2}"/>
+        </geometry>
+      </visual>
+      <collision>
+        <origin xyz="0 0 0" rpy="0 0 0"/>
+        <geometry>
+          <sphere radius="${caster_height/2}"/>
+        </geometry>
+      </collision>
+      <xacro:sphere_inertia m="1.0" r="${caster_height/2}"/>
+    </link>
+    <joint name="${prefix}_caster_joint" type="fixed">
+      <parent link="base_link"/>
+      <child link="${prefix}_caster_wheel"/>
+      <origin xyz="${x_offset} 0 ${-base_height/2 - (caster_height/2)}" rpy="0 0 0"/>
+    </joint>
+    <gazebo reference="${prefix}_caster_joint">
+      <preserveFixedJoint>true</preserveFixedJoint>
+    </gazebo>
+    <gazebo reference="${prefix}_caster_wheel">
+      <mu1>0.001</mu1>
+      <mu2>0.001</mu2>
+    </gazebo>
   </xacro:macro>
   <xacro:macro name="shark_base">
@@ -75,4 +106,6 @@
     <xacro:wheel prefix="left" reflect="1" />
     <xacro:wheel prefix="right" reflect="-1" />
+    <xacro:caster_wheel prefix="front" x_offset="${base_len/2 - 0.05}" />
+    <xacro:caster_wheel prefix="rear" x_offset="${-base_len/2 + 0.05}" />
   </xacro:macro>
 </robot>
