Commit message: :bug: neck: camera on head_pan/head_tilt joints and attach camera driver frames
- Drive the camera chain with head_pan_joint / head_tilt_joint (camera pan/tilt
  motors, ids 8/9) instead of horizontal/vertical_neck_joint (animatronic head,
  ids 61/62). Restores the legacy link names head_pan_link / head_tilt_link
  used by the RViz configs. camera_link / camera_link_static unchanged.
- Add fixed joints camera_link -> femtobolt_link and camera_link -> realsense_link
  (zero offset). Since camera.launch.py switched camera_name from 'camera' to
  femtobolt/realsense (2026-04), the driver trees were no longer connected to
  the robot TF tree.

File: urdf/neck/neck.xacro (robot description, xacro)
@@ -2,10 +2,15 @@
 <!--
   BORIS neck + camera mount.
-  Joint names match what fbot_hri/fbot_head `neck_controller` publishes on
-  /boris_head/joint_states, so robot_state_publisher moves these joints directly:
-    horizontal_neck_joint  (pan,  about z)
-    vertical_neck_joint    (tilt, about y)
+  fbot_hri/fbot_head `neck_controller` drives four Dynamixels from one command
+  and publishes all of them on /boris_head/joint_states:
+    head_pan_joint         (id 8,  about z)  camera pan   <- modeled here
+    head_tilt_joint        (id 9,  about y)  camera tilt  <- modeled here
+    horizontal_neck_joint  (id 62)           animatronic head (face), left/right
+    vertical_neck_joint    (id 61)           animatronic head (face), up/down
+  The camera sits on the pan/tilt motors, so only those move camera_link.
+  The head motors follow the same command but carry no frame we use, so they
+  are not modeled (their joint states are ignored by robot_state_publisher).
   Frames (parent -> child):
-    <parent> -> neck_pan_link -> camera_mount_link -> camera_link
+    <parent> -> head_pan_link -> head_tilt_link -> camera_link
   A second, FIXED copy of the chain ends at `camera_link_static`. It does not
   follow the neck and is used as a reference frame (neck_controller default
@@ -28,5 +33,5 @@
   <xacro:macro name="neck" params="parent xyz rpy">
     <!-- Moving chain -->
-    <link name="neck_pan_link">
+    <link name="head_pan_link">
       <xacro:neck_part_inertial m="0.018"/>
       <visual>
@@ -38,5 +43,5 @@
       </collision>
     </link>
-    <link name="camera_mount_link">
+    <link name="head_tilt_link">
       <xacro:neck_part_inertial m="0.055"/>
       <visual>
@@ -58,15 +63,15 @@
       </collision>
     </link>
-    <joint name="horizontal_neck_joint" type="revolute">
+    <joint name="head_pan_joint" type="revolute">
       <origin xyz="${xyz}" rpy="${rpy}"/>
       <parent link="${parent}"/>
-      <child link="neck_pan_link"/>
+      <child link="head_pan_link"/>
       <axis xyz="0 0 1"/>
       <limit effort="1" lower="-1.57" upper="1.57" velocity="1"/>
     </joint>
-    <joint name="vertical_neck_joint" type="revolute">
+    <joint name="head_tilt_joint" type="revolute">
       <origin xyz="0 0 0.05" rpy="0 0 0"/>
-      <parent link="neck_pan_link"/>
-      <child link="camera_mount_link"/>
+      <parent link="head_pan_link"/>
+      <child link="head_tilt_link"/>
       <axis xyz="0 1 0"/>
       <limit effort="1" lower="-1.57" upper="1.57" velocity="1"/>
@@ -74,24 +79,42 @@
     <joint name="camera_joint" type="fixed">
       <origin xyz="0.06705 0 -0.00425" rpy="0 0 0"/>
-      <parent link="camera_mount_link"/>
+      <parent link="head_tilt_link"/>
       <child link="camera_link"/>
     </joint>
+    <!-- Camera drivers: each publishes its own tree rooted at <camera_name>_link
+         (fbot_bringup/camera.launch.py: camera_name femtobolt / realsense).
+         Attach both roots to camera_link so point clouds and detections follow
+         the pan/tilt. Zero offset = the pre-2026-04 setup, where camera_name was
+         'camera' and the driver root WAS camera_link. Only one camera runs at a
+         time; the other frame is simply unused. -->
+    <link name="femtobolt_link"/>
+    <joint name="femtobolt_joint" type="fixed">
+      <origin xyz="0 0 0" rpy="0 0 0"/>
+      <parent link="camera_link"/>
+      <child link="femtobolt_link"/>
+    </joint>
+    <link name="realsense_link"/>
+    <joint name="realsense_joint" type="fixed">
+      <origin xyz="0 0 0" rpy="0 0 0"/>
+      <parent link="camera_link"/>
+      <child link="realsense_link"/>
+    </joint>
     <!-- Fixed reference chain (does not follow the neck) -->
-    <link name="neck_pan_link_static"/>
-    <link name="camera_mount_link_static"/>
+    <link name="head_pan_link_static"/>
+    <link name="head_tilt_link_static"/>
     <link name="camera_link_static"/>
-    <joint name="neck_pan_joint_static" type="fixed">
+    <joint name="head_pan_joint_static" type="fixed">
       <origin xyz="${xyz}" rpy="${rpy}"/>
       <parent link="${parent}"/>
-      <child link="neck_pan_link_static"/>
+      <child link="head_pan_link_static"/>
     </joint>
-    <joint name="camera_mount_joint_static" type="fixed">
+    <joint name="head_tilt_joint_static" type="fixed">
       <origin xyz="0 0 0.05" rpy="0 0 0"/>
-      <parent link="neck_pan_link_static"/>
-      <child link="camera_mount_link_static"/>
+      <parent link="head_pan_link_static"/>
+      <child link="head_tilt_link_static"/>
     </joint>
     <joint name="camera_joint_static" type="fixed">
       <origin xyz="0.06705 0 -0.00425" rpy="0 0 0"/>
-      <parent link="camera_mount_link_static"/>
+      <parent link="head_tilt_link_static"/>
       <child link="camera_link_static"/>
     </joint>
