Commit message: :sparkles: BORIS v2 model from the Onshape CAD; versions selected by robot_version
- tools/v2_from_onshape.py: reads the Onshape URDF export, finds the wheel disks
  (r 0.0984, sep 0.344), rebuilds the neutral neck pose, writes decimated meshes
  (meshes/v2, ~1 MB) and config/robot/v2.yaml (base, torso, sensors, neck, arm mount,
  footprint). Deterministic; raw export stays outside git.
- config/base -> config/robot (base_version -> robot_version); the Nav2 footprint
  moves into config/robot/<v>.yaml.
- urdf: boris.urdf.xacro = base + urdf/<robot_version>/robot.xacro. v1 files moved to
  urdf/v1 (expanded URDF identical to before for all flag combinations); v2 reads every
  pose from the yaml, neck with head_pan/head_tilt joints and femtobolt_link.
- base.xacro: optional base.center_x and base.visual_mesh; hokuyo macro: mesh param.
- tests iterate robot versions; docs/v2_from_onshape.md (workflow, assumptions, open items).

File: urdf/base/base.xacro (robot description, xacro)
@@ -1,10 +1,12 @@
 <?xml version="1.0"?>
 <!--
-  BORIS differential-drive base (the "Shark" hoverboard base), parametrized by base_version.
-  Geometry comes ONLY from config/base/<base_version>.yaml. Do not hardcode
+  BORIS differential-drive base (the "Shark" hoverboard base), parametrized by robot_version.
+  Geometry comes ONLY from config/robot/<robot_version>.yaml. Do not hardcode
   dimensions here. Usage:
     <xacro:include filename="$(find fbot_description)/urdf/base/base.xacro" />
     <xacro:fbot_base/>
-  and pass base_version:=v1|v2 to xacro (default v1).
+  and pass robot_version:=v1|v2 to xacro (default v1). Optional keys in the yaml:
+  base.center_x     base box centre ahead (+) / behind (-) the wheel axle   [default 0]
+  base.visual_mesh  mesh for the base visual (collision stays a box)      [default: box]
   Frames: base_footprint -> base_link -> left_wheel / right_wheel.
   Joints: left_wheel_joint / right_wheel_joint (same names as ros2_control
@@ -12,6 +14,6 @@
 -->
 <robot xmlns:xacro="http://www.ros.org/wiki/xacro">
-  <xacro:arg name="base_version" default="v1"/>
-  <xacro:property name="base_cfg" value="${xacro.load_yaml('$(find fbot_description)/config/base/$(arg base_version).yaml')}"/>
+  <xacro:arg name="robot_version" default="v1"/>
+  <xacro:property name="base_cfg" value="${xacro.load_yaml('$(find fbot_description)/config/robot/$(arg robot_version).yaml')}"/>
   <xacro:include filename="$(find fbot_description)/urdf/base/materials.xacro" />
   <xacro:property name="base_len"          value="${base_cfg['base']['length']}"/>
@@ -23,4 +25,5 @@
   <xacro:property name="wheel_x_offset"    value="${base_cfg['wheel']['x_offset']}"/>
   <xacro:property name="caster_height"     value="${base_cfg['caster_height']}"/>
+  <xacro:property name="base_center_x"     value="${base_cfg['base'].get('center_x', 0.0)}"/>
   <xacro:macro name="box_inertia" params="m w h d">
     <inertial>
@@ -53,11 +56,11 @@
       <xacro:cylinder_inertia m="10" r="${wheel_radius}" h="${wheel_width}"/>
     </link>
-    <!-- The wheel axle sits at z = wheel_radius above the ground:
-         base_link is at (base_height/2 + caster_height) above base_footprint. -->
+    <!-- The wheel axle sits at z = wheel_radius above the ground, under base_footprint:
+         base_link is (base_center_x, 0, base_height/2 + caster_height) from base_footprint. -->
     <joint name="${prefix}_wheel_joint" type="continuous">
       <axis xyz="0 1 0"/>
       <parent link="base_link"/>
       <child link="${prefix}_wheel"/>
-      <origin xyz="${wheel_x_offset} ${reflect * wheel_separation / 2} ${wheel_radius - caster_height - base_height/2}" rpy="0 0 0"/>
+      <origin xyz="${wheel_x_offset - base_center_x} ${reflect * wheel_separation / 2} ${wheel_radius - caster_height - base_height/2}" rpy="0 0 0"/>
     </joint>
   </xacro:macro>
@@ -69,5 +72,10 @@
         <material name="lightgray"/>
         <geometry>
-          <box size="${base_len} ${base_width} ${base_height}"/>
+          <xacro:if value="${'visual_mesh' in base_cfg['base']}">
+            <mesh filename="${base_cfg['base']['visual_mesh']}"/>
+          </xacro:if>
+          <xacro:unless value="${'visual_mesh' in base_cfg['base']}">
+            <box size="${base_len} ${base_width} ${base_height}"/>
+          </xacro:unless>
         </geometry>
       </visual>
@@ -79,5 +87,5 @@
     </link>
     <joint name="base_link_joint" type="fixed">
-      <origin xyz="0 0 ${base_height/2 + caster_height}" rpy="0 0 0"/>
+      <origin xyz="${base_center_x} 0 ${base_height/2 + caster_height}" rpy="0 0 0"/>
       <parent link="base_footprint"/>
       <child link="base_link"/>

File: urdf/base/base_ros2_control.xacro (robot description, xacro)
@@ -3,5 +3,5 @@
   ros2_control hardware description for the base (hoverboard_driver).
   Included by urdf/base/base.xacro, which defines the `base_cfg` property
-  (config/base/<base_version>.yaml). Do not include this file on its own.
+  (config/robot/<robot_version>.yaml). Do not include this file on its own.
 -->
 <robot xmlns:xacro="http://www.ros.org/wiki/xacro">

File: urdf/boris.urdf.xacro (robot description, xacro)
@@ -3,46 +3,21 @@
   BORIS robot description.
   xacro args:
-    base_version   v1 | v2    Shark base geometry (config/base/<v>.yaml)         [default v1]
-    use_neck       true|false neck + camera mount (urdf/neck/neck.xacro)         [default true]
+    robot_version  v1 | v2    which BORIS (config/robot/<v>.yaml, urdf/<v>/robot.xacro) [default v1]
+    use_neck       true|false neck + camera mount (urdf/<v>/neck.xacro)          [default true]
     use_arm_mount  true|false mounting plate the arm is attached to (no arm model)     [default true]
-    arm_z_position <m>        height of the plate on the torso                         [default 0.315]
+    arm_z_position <m>        v1: height of the plate on the torso                     [default 0.315]
     use_sick       true|false Sick LMS1xx mount                                        [default true]
-  Check it:  xacro boris.urdf.xacro base_version:=v1 | check_urdf /dev/stdin
+  Check it:  xacro boris.urdf.xacro robot_version:=v2 | check_urdf /dev/stdin
 -->
 <robot xmlns:xacro="http://www.ros.org/wiki/xacro" name="boris">
-  <xacro:arg name="base_version"   default="v1"/>
+  <xacro:arg name="robot_version"  default="v1"/>
   <xacro:arg name="use_neck"       default="true"/>
   <xacro:arg name="use_arm_mount"  default="true"/>
   <xacro:arg name="arm_z_position" default="0.315"/>
   <xacro:arg name="use_sick"       default="true"/>
-  <!-- Base (geometry from config/base/<base_version>.yaml) -->
+  <!-- Base: geometry from config/robot/<robot_version>.yaml (defines the base_cfg property) -->
   <xacro:include filename="$(find fbot_description)/urdf/base/base.xacro"/>
   <xacro:fbot_base/>
-  <!-- Body, sensors, neck -->
-  <xacro:include filename="$(find fbot_description)/urdf/body.xacro"/>
-  <xacro:include filename="$(find fbot_description)/urdf/sensors/hokuyo.xacro"/>
-  <xacro:include filename="$(find fbot_description)/urdf/sensors/sick_lms1xx.xacro"/>
-  <xacro:include filename="$(find fbot_description)/urdf/neck/neck.xacro"/>
-  <xacro:dorso parent="base_link"/>
-  <xacro:if value="$(arg use_arm_mount)">
-    <xacro:arm_mount parent="dorso_link" z="$(arg arm_z_position)"/>
-  </xacro:if>
-  <xacro:if value="$(arg use_neck)">
-    <xacro:neck parent="dorso_link" xyz="${dorso_len/2 + 0.05} 0 ${dorso_height + 0.053}" rpy="0 0 0"/>
-  </xacro:if>
-  <!-- Lasers (frame names must match config/sensors/urg_*.yaml) -->
-  <xacro:sensor_hokuyo parent="base_link" name="ground"
-      xyz="${base_len/2 + 0.017 + 0.024} 0 ${0.02 - base_height/2}" rpy="${pi} 0 0"/>
-  <xacro:sensor_hokuyo parent="base_link" name="back"
-      xyz="${-base_len/2 - 0.017 - 0.024} 0 ${0.02 - base_height/2}" rpy="${pi} 0 ${pi}"/>
-  <xacro:if value="$(arg use_sick)">
-    <xacro:sick_lms_1xx name="sick" ros_topic="/scan"/>
-    <joint name="laser_joint" type="fixed">
-      <origin xyz="${base_len/2 + 0.017 + 0.05} 0 ${0.02 + base_height/2}" rpy="0 0 0"/>
-      <parent link="base_link"/>
-      <child link="sick_mount_link"/>
-    </joint>
-  </xacro:if>
-  <!-- IMU (frame_id of the bno055 driver must be imu_link) -->
-  <xacro:imu parent="base_link" xyz="0 0.06 ${base_height/2 - 0.05}" rpy="${pi} 0 ${-pi/2}"/>
+  <!-- Body, sensors, neck of this robot version -->
+  <xacro:include filename="$(find fbot_description)/urdf/$(arg robot_version)/robot.xacro"/>
 </robot>

File: urdf/sensors/hokuyo.xacro (robot description, xacro)
@@ -2,5 +2,5 @@
 <robot name="sensor_hokuyo"
   xmlns:xacro="http://ros.org/wiki/xacro">
-  <xacro:macro name="sensor_hokuyo" params="parent xyz rpy name">
+  <xacro:macro name="sensor_hokuyo" params="parent xyz rpy name mesh:=package://fbot_description/meshes/sensors/hokuyo.dae">
     <link name="hokuyo_${name}_link">
       <!--collision>
@@ -13,5 +13,5 @@
         <origin xyz="0 0 0" rpy="0 0 0"/>
         <geometry>
-          <mesh filename="package://fbot_description/meshes/sensors/hokuyo.dae"/>
+          <mesh filename="${mesh}"/>
         </geometry>
       </visual>

File: urdf/v1/body.xacro (robot description, xacro)
@@ -3,5 +3,5 @@
   BORIS body: everything that sits on top of the Shark base.
   Requires urdf/base/base.xacro to be included first (it defines base_len,
-  base_height, ... from config/base/<base_version>.yaml).
+  base_height, ... from config/robot/<robot_version>.yaml).
   Frames: base_link -> dorso_link -> [arm_mount_link]
           base_link -> hokuyo_ground_link, hokuyo_back_link, sick_mount_link, imu_link

File: urdf/v1/neck.xacro (robot description, xacro)
@@ -17,5 +17,5 @@
   target_frame, infinite_rotate_camera state).
   Usage:
-    <xacro:include filename="$(find fbot_description)/urdf/neck/neck.xacro"/>
+    <xacro:include filename="$(find fbot_description)/urdf/v1/neck.xacro"/>
     <xacro:neck parent="dorso_link" xyz="..." rpy="0 0 0"/>
   NOTE: the facial joints (jaw, eyes, eyelids, eyebrows) are driven by
